Commit message: Added Gazebo Funcionality

File: description/robot_core.xacro (robot description, xacro)
@@ -33,5 +33,5 @@
             <material name="white"/>
         </visual>
-        <collison>
+        <collision>
             <origin xyz="0.15 0.0 0.075"/>
             <geometry>
@@ -39,9 +39,14 @@
             </geometry>
             <material name="white"/>
-        </collison>
+        </collision>
         <xacro:inertial_box mass="0.5" x="0.3" y="0.3" z="0.15">
             <origin xyz= "0.15 0.0 0.075" rpy="0.0 0.0 0.0"/>
         </xacro:inertial_box>
     </link>
+    <gazebo reference="chassis">
+        <material>
+            Gazebo/White
+        </material>
+    </gazebo>
     <!--Left Wheel-->
     <joint name="left_wheel_joint" type="continuous">
@@ -58,14 +63,19 @@
             <material name="blue"/>
         </visual>
-         <collison>
+        <collision>
             <geometry>
                 <cylinder radius="0.05" length="0.04"/>
             </geometry>
             <material name="blue"/>
-        </collison>
+        </collision>
         <xacro:inertial_cylinder mass="0.1" length="0.04" radius="0.05">
             <origin xyz= "0.0 0.0 0.0" rpy="0.0 0.0 0.0"/>
         </xacro:inertial_cylinder>
     </link>
+    <gazebo reference="left_wheel">
+        <material>
+            Gazebo/Blue
+        </material>
+    </gazebo>
      <!--Right Wheel-->
     <joint name="right_wheel_joint" type="continuous">
@@ -82,14 +92,19 @@
             <material name="blue"/>
         </visual>
-        <collison>
+        <collision>
             <geometry>
                 <cylinder radius="0.05" length="0.04"/>
             </geometry>
             <material name="blue"/>
-        </collison>
+        </collision>
         <xacro:inertial_cylinder mass="0.1" length="0.04" radius="0.05">
             <origin xyz= "0.0 0.0 0.0" rpy="0.0 0.0 0.0"/>
         </xacro:inertial_cylinder>
     </link>
+    <gazebo reference="right_wheel">
+        <material>
+            Gazebo/Blue
+        </material>
+    </gazebo>
     <!--Caster Wheel-->
     <joint name="caster_wheel_link" type="fixed">
@@ -105,13 +120,20 @@
             <material name="black"/>
         </visual>
-        <collison>
+        <collision>
             <geometry>
                 <sphere radius="0.05"/>
             </geometry>
             <material name="black"/>
-        </collison>
+        </collision>
         <xacro:inertial_sphere mass="0.1" radius="0.05">
             <origin xyz= "0.0 0.0 0.0" rpy="0.0 0.0 0.0"/>
         </xacro:inertial_sphere>
     </link>
+    <gazebo reference="caster_wheel">
+        <material>
+            Gazebo/Black
+        </material>
+        <mu1 value="0.01"/>
+        <mu2 value="0.01"/>
+    </gazebo>
 </robot>

Commit message: Added some new world

File: description/robot_core.xacro (robot description, xacro)
@@ -15,4 +15,7 @@
     <material name="black">
         <color rgba='0 0 0 1'/>
+    </material>
+    <material name="red">
+        <color rgba='1 0 0 1'/>
     </material>
      <!-- Base link -->
@@ -40,5 +43,5 @@
             <material name="white"/>
         </collision>
-        <xacro:inertial_box mass="0.5" x="0.3" y="0.3" z="0.15">
+        <xacro:inertial_box mass="1.5" x="0.3" y="0.3" z="0.15">
             <origin xyz= "0.15 0.0 0.075" rpy="0.0 0.0 0.0"/>
         </xacro:inertial_box>
